File: pwm.kicad_pcb (KiCad board)
At the start: 2 copper layers, 24.1 x 55.9 mm, 10 parts, among them Q1 IRF540N, U1 4069

Commit message: Add README, add preview images
Parts:
- C1: value C -> 0.033 uF
- R1, R2, R3: value R -> 1k
- R4: value R -> 50
Connections:
- U1 pad 14: (no net) -> +OUT
- U1 pad 7: (no net) -> Earth
Routing:
- net (no net): track 7.62 -> 0.00 mm
- net Earth: track 6.35 -> 11.4 mm
- net +OUT: track 0.00 -> 2.54 mm
Changed lines of the file:
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@@
     (zones 0)
     (modules 10)
-    (nets 14)
+    (nets 15)
   )
   (page A4)
@@
   (net 12 "Net-(RV1-Pad2)")
   (net 13 "Net-(U1-Pad2)")
+  (net 14 +OUT)
   (net_class Default "Это класс цепей по умолчанию."
     (clearance 0.2)
@@
     (uvia_dia 0.3)
     (uvia_drill 0.1)
+    (add_net +OUT)
     (add_net -OUT)
     (add_net Earth)
@@
       (effects (font (size 1 1) (thickness 0.15)))
     )
-    (fp_text value R (at 5.08 2.37 270) (layer F.Fab)
+    (fp_text value 1k (at 5.08 2.37 270) (layer F.Fab)
       (effects (font (size 1 1) (thickness 0.15)))
     )
@@
       (effects (font (size 1 1) (thickness 0.15)))
     )
-    (fp_text value R (at 5.08 2.37 180) (layer F.Fab)
+    (fp_text value 50 (at 5.08 2.37 180) (layer F.Fab)
       (effects (font (size 1 1) (thickness 0.15)))
     )
@@
       (effects (font (size 1 1) (thickness 0.15)))
     )
-    (fp_text value R (at 5.08 2.37) (layer F.Fab)
+    (fp_text value 1k (at 5.08 2.37) (layer F.Fab)
       (effects (font (size 1 1) (thickness 0.15)))
     )
@@
       (effects (font (size 1 1) (thickness 0.15)))
     )
-    (fp_text value R (at 5.08 2.37) (layer F.Fab)
+    (fp_text value 1k (at 5.08 2.37) (layer F.Fab)
       (effects (font (size 1 1) (thickness 0.15)))
     )
@@
       (effects (font (size 1 1) (thickness 0.15)))
     )
-    (fp_text value C (at 5 2.67 90) (layer F.Fab)
+    (fp_text value "0.033 uF" (at 5 2.67 90) (layer F.Fab)
       (effects (font (size 1 1) (thickness 0.15)))
     )
@@
     (pad 13 thru_hole oval (at 7.62 2.54) (size 2.4 1.6) (drill 0.8) (layers *.Cu *.Mask)
       (net 12 "Net-(RV1-Pad2)"))
-    (pad 7 thru_hole oval (at 0 15.24) (size 2.4 1.6) (drill 0.8) (layers *.Cu *.Mask))
-    (pad 14 thru_hole oval (at 7.62 0) (size 2.4 1.6) (drill 0.8) (layers *.Cu *.Mask))
+    (pad 7 thru_hole oval (at 0 15.24) (size 2.4 1.6) (drill 0.8) (layers *.Cu *.Mask)
+      (net 7 Earth))
+    (pad 14 thru_hole oval (at 7.62 0) (size 2.4 1.6) (drill 0.8) (layers *.Cu *.Mask)
+      (net 14 +OUT))
     (model ${KISYS3DMOD}/Package_DIP.3dshapes/DIP-14_W7.62mm.wrl
       (at (xyz 0 0 0))
@@
     (arrow2b (pts (xy 109.22 121.92) (xy 110.346504 121.333579)))
   )
-  (segment (start 124.46 86.36) (end 124.46 83.82) (width 0.25) (layer B.Cu) (net 0))
-  (segment (start 116.84 101.6) (end 111.76 101.6) (width 0.25) (layer B.Cu) (net 0))
   (segment (start 111.76 96.52) (end 116.84 96.52) (width 0.25) (layer B.Cu) (net 1))
   (segment (start 116.84 96.52) (end 116.84 93.98) (width 0.25) (layer B.Cu) (net 1))
@@
   (segment (start 120.65 109.22) (end 124.46 105.41) (width 0.25) (layer B.Cu) (net 6))
   (segment (start 124.46 105.41) (end 129.54 105.41) (width 0.25) (layer B.Cu) (net 6))
+  (segment (start 116.84 101.6) (end 111.76 101.6) (width 0.25) (layer B.Cu) (net 7))
   (segment (start 118.11 113.03) (end 115.57 113.03) (width 0.25) (layer B.Cu) (net 7))
   (segment (start 115.57 113.03) (end 111.76 113.03) (width 0.25) (layer B.Cu) (net 7))
@@
   (segment (start 119.38 99.06) (end 120.65 97.79) (width 0.25) (layer B.Cu) (net 12))
   (segment (start 116.84 88.9) (end 116.84 91.44) (width 0.25) (layer B.Cu) (net 13))
+  (segment (start 124.46 86.36) (end 124.46 83.82) (width 0.25) (layer B.Cu) (net 14))
   (zone (net 7) (net_name Earth) (layer B.Cu) (hatch edge 0.508)
     (connect_pads (clearance 0.508))
